File: projects/sensor_data_logger/electronics/generated/kicad/sensor_data_logger.kicad_pcb (KiCad board)
At the start: 2 copper layers, 70 x 50 mm, 18 parts, among them J1 USB-C POWER, J2 UART DEBUG, Q1 Ideal Diode, U1 ESP32-S3-WROOM-1, U2 ICM-42688-P, U3 3V3 Buck

Commit message: chore: regenerate sensor data logger artifacts
Regenerate electronics, mechanical, firmware, and validation outputs against the
UART debug connector, the fuse placement fix, and the 3D review preview. Adds the
3D-model-bearing KiCad board, the routed project files, and the new gate reports
(cross-domain consistency, mechanical connector cutouts/retention, mounting
integrity, DC operating point, power integrity, candidate critic, release).
Parts:
- added R5: 5K1 USB-C Rd, Resistor_SMD:R_0603_1608Metric, F.Cu at (22.0, 7.00)
- added R6: 5K1 USB-C Rd, Resistor_SMD:R_0603_1608Metric, F.Cu at (26.0, 7.00)
- C1, C2: footprint C0603 -> Capacitor_SMD:C_0603_1608Metric
- C9: footprint C1206 -> Capacitor_SMD:C_1206_3216Metric
- D1, Q1: footprint SOT23-6 -> Package_TO_SOT_SMD:SOT-23-6
- F1: footprint MIDI -> HW_Curated:MIDI_Fuse
- J1: footprint USB_C_16Pin -> Connector_USB:USB_C_GCT_USB4105
- J2: footprint Cortex_Debug_10Pin -> Connector_Samtec:FTSH-105
- R1, R2, R3: footprint R0603 -> Resistor_SMD:R_0603_1608Metric
- U2: footprint LGA14 -> Package_LGA:LGA-14
- U3: footprint VQFN16 -> Package_DFN_QFN:VQFN-16
- moved J2 6.40 mm to (54.0, 39.0)
- moved F1 6.00 mm to (26.0, 10.0)
- moved U1 1.00 mm to (44.0, 43.0)
Routing:
- net V3V3: track 109.0 -> 95.0 mm
- net UART_RX: track 18.1 -> 28.1 mm
- net USB_CC1: track 0.00 -> 9.36 mm
- net I2C_IMU_SCL: track 50.2 -> 42.3 mm
- net USB_DP: track 52.0 -> 44.5 mm, vias 1 -> 0
- net USB_DM_RAW: track 12.5 -> 17.7 mm
- net I2C_IMU_SDA: track 41.6 -> 46.1 mm, vias 0 -> 1
- net GND: track 142.0 -> 146.0 mm
- net USB_CC2: track 0.00 -> 3.83 mm
- net UART_TX: track 13.8 -> 10.5 mm
- net BOOT: track 22.4 -> 19.2 mm
- net USB_DM: track 42.5 -> 39.7 mm, vias 1 -> 0
- net USB_FUSED: track 6.00 -> 8.49 mm
- net USB_VBUS: track 8.60 -> 10.5 mm
- net IMU_INT: track 46.2 -> 44.8 mm
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- added copper zone on F.Cu, net GND
